File: Hardware/E-Bike_V2/E-Bike.kicad_pcb (KiCad board)
At the start: 2 copper layers, 36.3 x 26.5 mm, 38 parts, among them J1 AVR-ISP-6, J2 Conn_01x04, J3 Conn_01x02, J4 Conn_01x02, U1 MAX17552AUB+, U2 ATtiny85-20SU, U3 TPS76350, U4 INA290

Commit message: v2 hardware and added arduino PID with current sense sketch
Parts:
- added J5: Conn_01x04, Connector_PinHeader_2.54mm:PinHeader_1x04_P2.54mm_Vertical, F.Cu at (106.5, 114.5)
- added J6: Conn_01x04, Connector_PinHeader_2.54mm:PinHeader_1x04_P2.54mm_Vertical, F.Cu at (126.2, 114.5)
Connections:
- net Net-(R2-Pad1) renamed /VBUS_R
Routing:
- net +10V: track 11.8 -> 22.6 mm, vias 2 -> 3

Commit message: updated algo for v2, started v3 design
Other:
- net class Default removed
